File: HARDWARE/A64-OLinuXino/A64-OlinuXino_Rev_A/A64-OlinuXino_Rev_A.sch (KiCad schematic (older format))
At the start: 50 parts, among them U1 AllWinner-A64(FBGA396), U2 K4B4G1646D-BCK0(FBGA-96_256Mx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, U3 K4B4G1646D-BCK0(FBGA-96_256Mx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

Commit message: A64-OLinuXino component placement, all components libraries updated
Parts:
- U1: footprint (none) -> OLIMEX_IC-FP:FBGA396
- U2, U3: footprint (none) -> OLIMEX_IC-FP:FBGA96(HYNIX_SAMSUNG_512MX16_DDR3)
- renumbered C13 to C1, C32 to C10, C10 to C11, C14 to C12, C16 to C13, C18 to C14, C20 to C15, C22 to C16, C25 to C17, C27 to C18, C29 to C19, C15 to C2, C31 to C20, C33 to C21, C8 to C22, C11 to C23, C12 to C24, C23 to C25, C1 to C26, C2 to C27, C3 to C28, C4 to C29, C17 to C3, C5 to C30, C6 to C31, C7 to C32, C9 to C33, C19 to C4, C21 to C5, C24 to C6, C26 to C7, C28 to C8, C30 to C9, R10 to R1, R13 to R10, R1 to R11, R5 to R12, R9 to R13, R11 to R2, R2 to R3, R3 to R4, R6 to R5, R12 to R6, R4 to R7, R7 to R8, R8 to R9

Commit message: A64-OLinuXino update
Parts:
- R1, R10, R11, R12, R13, R14, R5, R6, R7, R8, R9: footprint OLIMEX_RLC-FP:R_0603_5MIL_DWS -> OLIMEX_RLC-FP:R_0402_5MIL_DWS
Connections:
- net S0SDQ0: now also U2.F7 (DQL1); no longer U2.E3 (DQL0)
- net S0SDQ1: now also U2.G2 (DQL6); no longer U2.F7 (DQL1)
- net S0SDQ10: now also U2.B8 (DQU6); no longer U2.C8 (DQU2)
- net S0SDQ11: now also U2.D7 (DQU0); no longer U2.C2 (DQU3)
- net S0SDQ12: now also U2.A3 (DQU7); no longer U2.A7 (DQU4)
- net S0SDQ13: now also U2.C2 (DQU3); no longer U2.A2 (DQU5)
- net S0SDQ14: now also U2.C3 (DQU1); no longer U2.B8 (DQU6)
- net S0SDQ15: now also U2.A2 (DQU5); no longer U2.A3 (DQU7)
- net S0SDQ16: now also U3.F7 (DQL1); no longer U3.E3 (DQL0)
- net S0SDQ17: now also U3.H8 (DQL5); no longer U3.F7 (DQL1)
- net S0SDQ18: now also U3.H7 (DQL7); no longer U3.F2 (DQL2)
- net S0SDQ21: now also U3.F2 (DQL2); no longer U3.H8 (DQL5)
- net S0SDQ22: now also U3.E3 (DQL0); no longer U3.G2 (DQL6)
- net S0SDQ23: now also U3.G2 (DQL6); no longer U3.H7 (DQL7)
- net S0SDQ24: now also U3.A7 (DQU4); no longer U3.D7 (DQU0)
- net S0SDQ25: now also U3.C8 (DQU2); no longer U3.C3 (DQU1)
- net S0SDQ26: now also U3.D7 (DQU0); no longer U3.C8 (DQU2)
- net S0SDQ27: now also U3.B8 (DQU6); no longer U3.C2 (DQU3)
- net S0SDQ28: now also U3.A3 (DQU7); no longer U3.A7 (DQU4)
- net S0SDQ29: now also U3.C3 (DQU1); no longer U3.A2 (DQU5)
- net S0SDQ3: now also U2.H7 (DQL7); no longer U2.F8 (DQL3)
- net S0SDQ30: now also U3.A2 (DQU5); no longer U3.B8 (DQU6)
- net S0SDQ31: now also U3.C2 (DQU3); no longer U3.A3 (DQU7)
- net S0SDQ4: now also U2.E3 (DQL0); no longer U2.H3 (DQL4)
- net S0SDQ5: now also U2.H3 (DQL4); no longer U2.H8 (DQL5)
- net S0SDQ6: now also U2.H8 (DQL5); no longer U2.G2 (DQL6)
- net S0SDQ7: now also U2.F8 (DQL3); no longer U2.H7 (DQL7)
- net S0SDQ8: now also U2.A7 (DQU4); no longer U2.D7 (DQU0)
- net S0SDQ9: now also U2.C8 (DQU2); no longer U2.C3 (DQU1)
- net S0SCKN renamed S0SCK_N
- net S0SCKP renamed S0SCK_P
- net S0SDQS0N renamed S0SDQS0_N
- net S0SDQS0P renamed S0SDQS0_P
- net S0SDQS1N renamed S0SDQS1_N
- net S0SDQS1P renamed S0SDQS1_P
- net S0SDQS2N renamed S0SDQS2_N
- net S0SDQS2P renamed S0SDQS2_P
- net S0SDQS3N renamed S0SDQS3_N
- net S0SDQS3P renamed S0SDQS3_P
Changed lines of the file:
@@
 EESchema Schematic File Version 2
-LIBS:OLIMEX_Antennas
-LIBS:OLIMEX_Buttons
-LIBS:OLIMEX_Connectors
-LIBS:OLIMEX_Devices
-LIBS:OLIMEX_Diodes
-LIBS:OLIMEX_IC
-LIBS:OLIMEX_Jumpers
-LIBS:OLIMEX_OTHER
-LIBS:OLIMEX_Power
-LIBS:OLIMEX_RCL
-LIBS:OLIMEX_Regulators
-LIBS:OLIMEX_Switches
-LIBS:OLIMEX_Transistors
 LIBS:A64-OlinuXino_Rev_A-cache
 EELAYER 25 0
@@
 F 0 "R7" H 4525 7550 50  0000 C CNN
 F 1 "243R/1%" H 4050 7550 50  0000 C CNN
-F 2 "OLIMEX_RLC-FP:R_0603_5MIL_DWS" V 4280 7600 30  0001 C CNN
+F 2 "OLIMEX_RLC-FP:R_0402_5MIL_DWS" V 4280 7600 30  0001 C CNN
 F 3 "" H 4350 7600 30  0000 C CNN
 	1    4350 7600
@@
 S0SBA2
 Text Label 4300 5000 0    60   ~ 0
-S0SCKP
+S0SCK_P
 Text Label 4300 5100 0    60   ~ 0
-S0SCKN
+S0SCK_N
 Text Label 4300 5200 0    60   ~ 0
 S0SCKE0
@@
 S0SBA2
 Text Label 7700 4500 0    60   ~ 0
-S0SCKP
+S0SCK_P
 Text Label 7700 4600 0    60   ~ 0
-S0SCKN
+S0SCK_N
 Text Label 7700 4700 0    60   ~ 0
 S0SCKE0
@@
 S0SDQM3
 Text Label 4300 5900 0    60   ~ 0
-S0SDQS0P
+S0SDQS0_P
 Text Label 4300 6000 0    60   ~ 0
-S0SDQS0N
+S0SDQS0_N
 Text Label 4300 6100 0    60   ~ 0
-S0SDQS1P
+S0SDQS1_P
 Text Label 4300 6200 0    60   ~ 0
-S0SDQS1N
+S0SDQS1_N
 Text Label 4300 6300 0    60   ~ 0
-S0SDQS2P
+S0SDQS2_P
 Text Label 4300 6400 0    60   ~ 0
-S0SDQS2N
+S0SDQS2_N
 Text Label 4300 6500 0    60   ~ 0
-S0SDQS3P
+S0SDQS3_P
 Text Label 4300 6600 0    60   ~ 0
-S0SDQS3N
+S0SDQS3_N
 Text Label 4300 6700 0    60   ~ 0
 S0SCS0
@@
 S0SDQM1
 Text Label 7700 5300 0    60   ~ 0
-S0SDQS1P
+S0SDQS1_P
 Text Label 7700 5400 0    60   ~ 0
-S0SDQS1N
+S0SDQS1_N
 Text Label 7700 5600 0    60   ~ 0
-S0SDQS0P
+S0SDQS0_P
 Text Label 7700 5700 0    60   ~ 0
-S0SDQS0N
+S0SDQS0_N
 Text Label 7700 5900 0    60   ~ 0
 S0SCS0
@@
 Text Label 7700 6700 0    60   ~ 0
 S0SODT1
-Text Label 9400 3900 0    60   ~ 0
+Text Label 9400 3800 0    60   ~ 0
 S0SDQ0
-Text Label 9400 3800 0    60   ~ 0
+Text Label 9400 3300 0    60   ~ 0
 S0SDQ1
 Text Label 9400 3700 0    60   ~ 0
 S0SDQ2
+Text Label 9400 3200 0    60   ~ 0
+S0SDQ3
+Text Label 9400 3900 0    60   ~ 0
+S0SDQ4
+Text Label 9400 3500 0    60   ~ 0
+S0SDQ5
+Text Label 9400 3400 0    60   ~ 0
+S0SDQ6
 Text Label 9400 3600 0    60   ~ 0
-S0SDQ3
-Text Label 9400 3500 0    60   ~ 0
-S0SDQ4
-Text Label 9400 3400 0    60   ~ 0
-S0SDQ5
-Text Label 9400 3300 0    60   ~ 0
-S0SDQ6
-Text Label 9400 3200 0    60   ~ 0
 S0SDQ7
+Text Label 9400 2700 0    60   ~ 0
+S0SDQ8
+Text Label 9400 2900 0    60   ~ 0
+S0SDQ9
+Text Label 9400 2500 0    60   ~ 0
+S0SDQ10
 Text Label 9400 3100 0    60   ~ 0
-S0SDQ8
+S0SDQ11
+Text Label 9400 2400 0    60   ~ 0
+S0SDQ12
+Text Label 9400 2800 0    60   ~ 0
+S0SDQ13
 Text Label 9400 3000 0    60   ~ 0
-S0SDQ9
-Text Label 9400 2900 0    60   ~ 0
-S0SDQ10
-Text Label 9400 2800 0    60   ~ 0
-S0SDQ11
-Text Label 9400 2700 0    60   ~ 0
-S0SDQ12
+S0SDQ14
 Text Label 9400 2600 0    60   ~ 0
-S0SDQ13
-Text Label 9400 2500 0    60   ~ 0
-S0SDQ14
-Text Label 9400 2400 0    60   ~ 0
 S0SDQ15
 $Comp
@@
 F 0 "R9" H 7800 8050 50  0000 C CNN
 F 1 "243R/1%" H 7300 8050 50  0000 C CNN
-F 2 "OLIMEX_RLC-FP:R_0603_5MIL_DWS" V 7530 8100 30  0001 C CNN
+F 2 "OLIMEX_RLC-FP:R_0402_5MIL_DWS" V 7530 8100 30  0001 C CNN
 F 3 "" H 7600 8100 30  0000 C CNN
 	1    7600 8100
@@
 F 0 "R13" H 7800 8150 50  0000 C CNN
 F 1 "NA(243R/1%)" H 7200 8150 50  0000 C CNN
-F 2 "OLIMEX_RLC-FP:R_0603_5MIL_DWS" V 7530 8200 30  0001 C CNN
+F 2 "OLIMEX_RLC-FP:R_0402_5MIL_DWS" V 7530 8200 30  0001 C CNN
 F 3 "" H 7600 8200 30  0000 C CNN
 	1    7600 8200
@@
 F 0 "R8" V 7250 7850 50  0000 C CNN
 F 1 "2k/1%" V 7150 7925 50  0000 C CNN
-F 2 "OLIMEX_RLC-FP:R_0603_5MIL_DWS" V 7130 7750 30  0001 C CNN
+F 2 "OLIMEX_RLC-FP:R_0402_5MIL_DWS" V 7130 7750 30  0001 C CNN
 F 3 "" H 7200 7750 30  0000 C CNN
 	1    7200 7750
@@
 F 0 "R5" V 7250 7250 50  0000 C CNN
 F 1 "2k/1%" V 7150 7325 50  0000 C CNN
-F 2 "OLIMEX_RLC-FP:R_0603_5MIL_DWS" V 7130 7150 30  0001 C CNN
+F 2 "OLIMEX_RLC-FP:R_0402_5MIL_DWS" V 7130 7150 30  0001 C CNN
 F 3 "" H 7200 7150 30  0000 C CNN
 	1    7200 7150
@@
 F 0 "R12" H 4700 8150 50  0000 C CNN
 F 1 "2k/1%" H 4300 8150 50  0000 C CNN
-F 2 "OLIMEX_RLC-FP:R_0603_5MIL_DWS" V 4480 8200 30  0001 C CNN
+F 2 "OLIMEX_RLC-FP:R_0402_5MIL_DWS" V 4480 8200 30  0001 C CNN
 F 3 "" H 4550 8200 30  0000 C CNN
 	1    4550 8200
@@
 F 0 "R11" H 3900 8150 50  0000 C CNN
 F 1 "2k/1%" H 3500 8150 50  0000 C CNN
-F 2 "OLIMEX_RLC-FP:R_0603_5MIL_DWS" V 3680 8200 30  0001 C CNN
+F 2 "OLIMEX_RLC-FP:R_0402_5MIL_DWS" V 3680 8200 30  0001 C CNN
 F 3 "" H 3750 8200 30  0000 C CNN
 	1    3750 8200
@@
 S0SBA2
 Text Label 13100 4500 0    60   ~ 0
-S0SCKP
+S0SCK_P
 Text Label 13100 4600 0    60   ~ 0
-S0SCKN
+S0SCK_N
 Text Label 13100 4700 0    60   ~ 0
 S0SCKE0
@@
 S0SDQM3
 Text Label 13100 5300 0    60   ~ 0
-S0SDQS3P
+S0SDQS3_P
 Text Label 13100 5400 0    60   ~ 0
-S0SDQS3N
+S0SDQS3_N
 Text Label 13100 5600 0    60   ~ 0
-S0SDQS2P
+S0SDQS2_P
 Text Label 13100 5700 0    60   ~ 0
-S0SDQS2N
+S0SDQS2_N
 Text Label 13100 5900 0    60   ~ 0
 S0SCS0
@@
 F 0 "R10" H 13100 8050 50  0000 C CNN
 F 1 "243R/1%" H 12575 8050 50  0000 C CNN
-F 2 "OLIMEX_RLC-FP:R_0603_5MIL_DWS" V 12830 8100 30  0001 C CNN
+F 2 "OLIMEX_RLC-FP:R_0402_5MIL_DWS" V 12830 8100 30  0001 C CNN
 F 3 "" H 12900 8100 30  0000 C CNN
 	1    12900 8100
@@
 F 0 "R14" H 13100 8150 50  0000 C CNN
 F 1 "NA(243R/1%)" H 12500 8150 50  0000 C CNN
-F 2 "OLIMEX_RLC-FP:R_0603_5MIL_DWS" V 12830 8200 30  0001 C CNN
+F 2 "OLIMEX_RLC-FP:R_0402_5MIL_DWS" V 12830 8200 30  0001 C CNN
 F 3 "" H 12900 8200 30  0000 C CNN
 	1    12900 8200
@@
 	-1   0    0    -1
 $EndComp
-Text Label 15200 3900 2    60   ~ 0
+Text Label 15200 3800 2    60   ~ 0
 S0SDQ16
-Text Label 15200 3800 2    60   ~ 0
+Text Label 15200 3400 2    60   ~ 0
 S0SDQ17
-Text Label 15200 3700 2    60   ~ 0
+Text Label 15200 3200 2    60   ~ 0
 S0SDQ18
 Text Label 15200 3600 2    60   ~ 0
@@
 Text Label 15200 3500 2    60   ~ 0
 S0SDQ20
-Text Label 15200 3400 2    60   ~ 0
+Text Label 15200 3700 2    60   ~ 0
 S0SDQ21
+Text Label 15200 3900 2    60   ~ 0
+S0SDQ22
 Text Label 15200 3300 2    60   ~ 0
-S0SDQ22
-Text Label 15200 3200 2    60   ~ 0
 S0SDQ23
+Text Label 15200 2700 2    60   ~ 0
+S0SDQ24
+Text Label 15200 2900 2    60   ~ 0
+S0SDQ25
 Text Label 15200 3100 2    60   ~ 0
-S0SDQ24
+S0SDQ26
+Text Label 15200 2500 2    60   ~ 0
+S0SDQ27
+Text Label 15200 2400 2    60   ~ 0
+S0SDQ28
 Text Label 15200 3000 2    60   ~ 0
-S0SDQ25
-Text Label 15200 2900 2    60   ~ 0
-S0SDQ26
+S0SDQ29
+Text Label 15200 2600 2    60   ~ 0
+S0SDQ30
 Text Label 15200 2800 2    60   ~ 0
-S0SDQ27
-Text Label 15200 2700 2    60   ~ 0
-S0SDQ28
-Text Label 15200 2600 2    60   ~ 0
-S0SDQ29
-Text Label 15200 2500 2    60   ~ 0
-S0SDQ30
-Text Label 15200 2400 2    60   ~ 0
 S0SDQ31
 Wire Wire Line
@@
 	7100 5100 7000 5000
 Text Label 12200 4500 2    60   ~ 0
-S0SCKP
+S0SCK_P
 Text Label 12200 5000 2    60   ~ 0
-S0SCKN
+S0SCK_N
 Wire Wire Line
 	12300 4500 11800 4500
@@
 F 0 "R1" V 11850 3900 50  0000 C CNN
 F 1 "2k/1%" V 11750 3950 50  0000 C CNN
-F 2 "OLIMEX_RLC-FP:R_0603_5MIL_DWS" V 11730 3750 30  0001 C CNN
+F 2 "OLIMEX_RLC-FP:R_0402_5MIL_DWS" V 11730 3750 30  0001 C CNN
 F 3 "" H 11800 3750 30  0000 C CNN
 	1    11800 3750
@@
 F 0 "R6" V 12650 7000 50  0000 C CNN
 F 1 "NA" V 12550 7025 50  0000 C CNN
-F 2 "OLIMEX_RLC-FP:R_0603_5MIL_DWS" V 12530 7150 30  0001 C CNN
+F 2 "OLIMEX_RLC-FP:R_0402_5MIL_DWS" V 12530 7150 30  0001 C CNN
 F 3 "" H 12600 7150 30  0000 C CNN
 	1    12600 7150
