File: HARDWARE/STMP157-OLinuXino-LIME2/1. Latest hardware revision/STMP157-OLinuXino-LIME2_Rev_B1/HDMI, LCD  and Ethernet.sch (KiCad schematic (older format))
At the start: 97 parts, among them Q3 Q25MHz/20pF/20ppm/4P/3.2x2.5mm, U1 STM32MP157CAA3x, U4 KSZ9031RNXCC(QFN48_1DRILL(PAD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, U5 NA(RCLAMP0524P(SLP2510P8)), U6 NA(RCLAMP0524P(SLP2510P8)), U7 NA(RCLAMP0524P(SLP2510P8)), U8 IT66121FN, U9 AT24C16C-SSHM-T

Commit message: 3d view components fixed
Parts:
- 1.25_EXT1: symbol OLIMEX_OTHER:TESTPAD -> STMP157-OLinuXino-LIME2_Rev_B1:TESTPAD
- C123, C47, C48, C49, C50, C51, C52, C53, C54, C55, C56, C57, C58, C59, C60, C61, C62, C63, C64, C65, C66, C67, C68, C69, C70, C71, C72, C73, C74, C75, C76, C77, C78, C79, C80, C81, C82, C83, C84, C85: symbol OLIMEX_RCL:C -> STMP157-OLinuXino-LIME2_Rev_B1:C
- D1: symbol OLIMEX_Diodes:D -> STMP157-OLinuXino-LIME2_Rev_B1:D
- FUSE1: symbol OLIMEX_Devices:FSMD035 -> STMP157-OLinuXino-LIME2_Rev_B1:FSMD035
- HDMI1: symbol OLIMEX_Connectors:HDMI-SWM-19 -> STMP157-OLinuXino-LIME2_Rev_B1:HDMI-SWM-19
- L2, L3, L4, L5, L6, L7: symbol OLIMEX_RCL:L -> STMP157-OLinuXino-LIME2_Rev_B1:L
- LAN1: symbol OLIMEX_Connectors:TM211Q01FM22 -> STMP157-OLinuXino-LIME2_Rev_B1:TM211Q01FM22
- LCD_CON1: symbol OLIMEX_Connectors:LCD_CON -> STMP157-OLinuXino-LIME2_Rev_B1:LCD_CON
- Q3: symbol OLIMEX_Devices:Crystal_GND -> STMP157-OLinuXino-LIME2_Rev_B1:Crystal_GND
- R42, R57, R58, R59, R60, R61, R62, R63, R64, R65, R66, R67, R68, R69, R70, R71, R72, R73, R74, R75, R76, R77, R78, R80, R81, R82, R87, R88, R89, R90, R91, R92, R93: symbol OLIMEX_RCL:R -> STMP157-OLinuXino-LIME2_Rev_B1:R
- RM2, RM3, RM4: symbol OLIMEX_RCL:RA1206_(4x0603)_4B8_Smashed -> STMP157-OLinuXino-LIME2_Rev_B1:RA1206_(4x0603)_4B8_Smashed
- U1: symbol OLIMEX_IC:STM32MP157CAA3x -> STMP157-OLinuXino-LIME2_Rev_B1:STM32MP157CAA3x
- U4: symbol OLIMEX_IC:KSZ9031RNXCC(QFN48_1DRILL(PADPITCH-0.5MM)) -> STMP157-OLinuXino-LIME2_Rev_B1:KSZ9031RNXCC(QFN48_1DRILL(PADPITCH-0.5MM))
- U5, U6, U7: symbol OLIMEX_Devices:RCLAMP0524P -> STMP157-OLinuXino-LIME2_Rev_B1:RCLAMP0524P
- U8: symbol OLIMEX_IC:IT66121FN -> STMP157-OLinuXino-LIME2_Rev_B1:IT66121FN
- U9: symbol OLIMEX_IC:AT24C16BN-SH(SO-8_150mil) -> STMP157-OLinuXino-LIME2_Rev_B1:AT24C16BN-SH(SO-8_150mil)
- VR1: symbol OLIMEX_Regulators:AMS1117-ADJ -> STMP157-OLinuXino-LIME2_Rev_B1:AMS1117-ADJ
Other:
- note removed: "10k???"
- note removed: "Notes:\n1. Da se testva dali moze CEC liniqta da nqma pull-up, poneze v datasheet-a na IT66121FN pise, 4e ima vgradeno CEC PHY i vynsniq pull-up moze da pre4i!\nNa shemite na Radxa i BeagleBoneGreen ima, no na CX-919 modula merihme, 4e nqma! Da se testva i resi okon4atelno dali ste slagame ili ne!\n2. Dali da ne slozim PoE connectora na Etherneta + PoE modul optional???"
- note removed: "The schematic check is completed up to here!!!\nCheck again and the Flash-Header schematic!!!"
