File: HARDWARE/STMP157-OLinuXino-LIME2/1. Latest hardware revision/STMP157-OLinuXino-LIME2_Rev_B1/Power Supply.sch (KiCad schematic (older format))
At the start: 146 parts, among them T1 LMUN2211LT1G(SOT-23), U1 STM32MP157CAA3x, U10 MT3608(SOT23-6), U11 SY8089AAAC(SOT23-5), U17 SY8089AAAC(SOT23-5), U18 AXP209(QFN-48), U19 RT9026GFP(MSOP-10), U20 MCP121T475I-TT(SOT23-3)

Commit message: 3d view components fixed
Parts:
- +1.2V_HDMI1, +2.8V1, +5V_EXT1, 1.2V_VDDCORE1, 1.35V_DDR1, 3.3V1, GND1, IPS1, VBAT-RTC1, VBUS1, VDD-FLASH1, VDD_USB1: symbol OLIMEX_OTHER:TESTPAD -> STMP157-OLinuXino-LIME2_Rev_B1:TESTPAD
- 5V_E1: symbol OLIMEX_Jumpers:SJ -> STMP157-OLinuXino-LIME2_Rev_B1:SJ
- BACKUP1: symbol OLIMEX_Connectors:CON2 -> STMP157-OLinuXino-LIME2_Rev_B1:CON2
- C100, C101, C102, C103, C104, C105, C106, C107, C108, C109, C111, C112, C113, C114, C115, C116, C117, C118, C119, C120, C121, C124, C125, C126, C134, C135, C136, C137, C138, C139, C140, C141, C142, C143, C144, C145, C146, C147, C148, C149, C150, C151, C152, C153, C154, C155, C156, C157, C158, C159, C160, C161, C162, C163, C164, C165, C166, C167, C44, C86, C87, C88, C89, C90, C91, C92, C93, C94, C95, C96, C97, C98, C99: symbol OLIMEX_RCL:C -> STMP157-OLinuXino-LIME2_Rev_B1:C
- CHGLED1, PWRLED1: symbol OLIMEX_Diodes:LED -> STMP157-OLinuXino-LIME2_Rev_B1:LED
- D2: symbol OLIMEX_Diodes:D_Schottky -> STMP157-OLinuXino-LIME2_Rev_B1:D_Schottky
- D4: symbol OLIMEX_Diodes:SMBJ6.0A -> STMP157-OLinuXino-LIME2_Rev_B1:SMBJ6.0A
- FET2, FET4: symbol OLIMEX_Transistors:P-MOS+DIOD -> STMP157-OLinuXino-LIME2_Rev_B1:P-MOS+DIOD
- FET3: symbol OLIMEX_Transistors:N-MOS+DIOD -> STMP157-OLinuXino-LIME2_Rev_B1:N-MOS+DIOD
- FUSE2: symbol OLIMEX_Devices:FSMD035 -> STMP157-OLinuXino-LIME2_Rev_B1:FSMD035
- L10, L11, L12, L13, L17, L8, L9: symbol OLIMEX_RCL:L -> STMP157-OLinuXino-LIME2_Rev_B1:L
- LIPO_BAT1: symbol OLIMEX_Connectors:BAT_CON -> STMP157-OLinuXino-LIME2_Rev_B1:BAT_CON
- PWR1: symbol OLIMEX_Connectors:PWR-JAKPWR_JACK_UNI_MILLING -> STMP157-OLinuXino-LIME2_Rev_B1:PWR-JAKPWR_JACK_UNI_MILLING
- PWRON1, RESET1: symbol OLIMEX_Buttons:T1107A(6x3,8x2,5MM) -> STMP157-OLinuXino-LIME2_Rev_B1:T1107A(6x3,8x2,5MM)
- R100, R101, R102, R103, R104, R105, R106, R107, R108, R109, R110, R111, R112, R113, R115, R116, R128, R133, R134, R135, R136, R137, R138, R44, R45, R52, R79, R83, R97, R98, R99: symbol OLIMEX_RCL:R -> STMP157-OLinuXino-LIME2_Rev_B1:R
- T1: symbol OLIMEX_Transistors:DTC114YKA(SOT-23) -> STMP157-OLinuXino-LIME2_Rev_B1:DTC114YKA(SOT-23)
- U1: symbol OLIMEX_IC:STM32MP157CAA3x -> STMP157-OLinuXino-LIME2_Rev_B1:STM32MP157CAA3x
- U10: symbol OLIMEX_Regulators:MT3608(SOT23-6) -> STMP157-OLinuXino-LIME2_Rev_B1:MT3608(SOT23-6)
- U11, U17: symbol OLIMEX_IC:SY8009AAAC(SOT23-5) -> STMP157-OLinuXino-LIME2_Rev_B1:SY8009AAAC(SOT23-5)
- U18: symbol OLIMEX_IC:AXP209(QFN-48) -> STMP157-OLinuXino-LIME2_Rev_B1:AXP209(QFN-48)
- U19: symbol OLIMEX_IC:RT9026G(P)FP(MSOP-10) -> STMP157-OLinuXino-LIME2_Rev_B1:RT9026G(P)FP(MSOP-10)
- U20: symbol OLIMEX_IC:MCP120 -> STMP157-OLinuXino-LIME2_Rev_B1:MCP120
- VR2: symbol OLIMEX_Regulators:AP1231-3.3V(SOT23-5) -> STMP157-OLinuXino-LIME2_Rev_B1:AP1231-3.3V(SOT23-5)
Other:
- note removed: "Notes:\n=========\n1. Da se testva dali ste e neobhodimo da se slagat RC grupi na DCDC-tata \ni ako ne da se iztriqt izlisnite elementi za sledvastata reviziq!!!\n2. Da se testva dali VTT_REF zahranva dobre MCU i DDR chipovete i ako e OK,\nda se iztriqt delitelite, syotvetnite kondenzatori i da se okysqt 0R rezistorite.\n3. Da se resi, okon4atelno, otkyde ste se zahranva RT9026GFP(MSOP-10) i da s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"
