File: HARDWARE/STMP157-OLinuXino-LIME2/1. Latest hardware revision/STMP157-OLinuXino-LIME2_Rev_B1/STMP157-OLinuXino-LIME2_Rev_B1.sch (KiCad schematic (older format))
At the start: 89 parts, among them U1 STM32MP157CAA3x, U2 K4B4G1646D-BYK0, U3 K4B4G1646D-BYK0

Commit message: 3d view components fixed
Parts:
- C1, C10, C11, C12, C122, C13, C14, C15, C16, C17, C18, C186, C187, C188, C189, C19, C190, C2, C20, C21, C22, C23, C24, C25, C26, C27, C28, C29, C3, C30, C31, C32, C33, C34, C35, C36, C37, C38, C39, C4, C5, C6, C7, C8, C9: symbol OLIMEX_RCL:C -> STMP157-OLinuXino-LIME2_Rev_B1:C
- R1, R10, R11, R12, R13, R132, R14, R15, R16, R17, R18, R19, R2, R20, R21, R22, R23, R24, R25, R26, R27, R28, R29, R3, R30, R31, R32, R33, R34, R35, R36, R37, R38, R39, R4, R47, R5, R6, R7, R8, R9: symbol OLIMEX_RCL:R -> STMP157-OLinuXino-LIME2_Rev_B1:R
- U1: symbol OLIMEX_IC:STM32MP157CAA3x -> STMP157-OLinuXino-LIME2_Rev_B1:STM32MP157CAA3x
- U2, U3: symbol OLIMEX_IC:H5TQ2G63BFR_MEM4G16D3EABG-125--H5TC8G63AMR-PBA_K4B8G1646Q-MYK0(FBGA-96_512MX16_DDR3-1600_11-11-11) -> STMP157-OLinuXino-LIME2_Rev_B1:H5TQ2G63BFR_MEM4G16D3EABG-125--H5TC8G63AMR-PBA_K4B8G1646Q-MYK0(FBGA-96_512MX16_DDR3-1600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
Other:
- note removed: "Notes:\n======\n1. Seriinite rezistori 22R na S0SCK_P i S0SCK_N gi nqma na Shemite na ST! Da se ima v predvid, ako imame problemi s DDR pametite, i da se smenqt s 0R ako e neobhodimo!"
