File: HARDWARE/STMP157-OLinuXino-LIME2/1. Latest hardware revision/STMP157-OLinuXino-LIME2_Rev_B1/USB, CAN and Extensions.sch (KiCad schematic (older format))
At the start: 54 parts, among them U1 STM32MP157CAA3x, U12 SY6280AAC(SOT23-5), U13 SY6280AAC(SOT23-5), U14 SY6280AAC(SOT23-5), U15 SIT1050T(SOIC-8_150mil)

Commit message: 3d view components fixed
Parts:
- 3.3V/5.0V1: symbol OLIMEX_Jumpers:SJ2W_Closed(1-2) -> STMP157-OLinuXino-LIME2_Rev_B1:SJ2W_Closed(1-2)
- C168, C169, C170, C172, C173, C174, C175, C176, C178, C179, C180, C181, C182, C183, C184, C185: symbol OLIMEX_RCL:C -> STMP157-OLinuXino-LIME2_Rev_B1:C
- CAN1, DBG1: symbol OLIMEX_Connectors:CON3 -> STMP157-OLinuXino-LIME2_Rev_B1:CON3
- CAN_T1: symbol OLIMEX_Jumpers:SJ -> STMP157-OLinuXino-LIME2_Rev_B1:SJ
- D3: symbol OLIMEX_Diodes:D_Schottky -> STMP157-OLinuXino-LIME2_Rev_B1:D_Schottky
- GPIO-1, GPIO-2, GPIO-3: symbol OLIMEX_Connectors:BH40S -> STMP157-OLinuXino-LIME2_Rev_B1:BH40S
- GPIO4: symbol OLIMEX_Connectors:BH20S -> STMP157-OLinuXino-LIME2_Rev_B1:BH20S
- L14, L15, L16: symbol OLIMEX_RCL:L -> STMP157-OLinuXino-LIME2_Rev_B1:L
- LED1: symbol OLIMEX_Diodes:LED -> STMP157-OLinuXino-LIME2_Rev_B1:LED
- LIME2_PLATFORM1: symbol OLIMEX_Cases:LIME2_PLATFORM -> STMP157-OLinuXino-LIME2_Rev_B1:LIME2_PLATFORM
- R114, R117, R118, R119, R120, R121, R122, R123, R124, R125, R126, R129, R130, R131, R140, R41: symbol OLIMEX_RCL:R -> STMP157-OLinuXino-LIME2_Rev_B1:R
- U1: symbol OLIMEX_IC:STM32MP157CAA3x -> STMP157-OLinuXino-LIME2_Rev_B1:STM32MP157CAA3x
- U12, U13, U14: symbol OLIMEX_IC:SY6280AAC(SOT23-5) -> STMP157-OLinuXino-LIME2_Rev_B1:SY6280AAC(SOT23-5)
- U15: symbol OLIMEX_IC:SIT1050T(SOIC-8_150mil) -> STMP157-OLinuXino-LIME2_Rev_B1:SIT1050T(SOIC-8_150mil)
- USB-OTG1: symbol OLIMEX_Connectors:USB-MINI -> STMP157-OLinuXino-LIME2_Rev_B1:USB-MINI
- USB1, USB2: symbol OLIMEX_Connectors:USB_A_VERTICAL -> STMP157-OLinuXino-LIME2_Rev_B1:USB_A_VERTICAL
Other:
- note removed: "1. Pro4eti Global_Future_Changes!!!!\n2. Opravi valutata na vsi4ki kondenzatori i rezistori\n3. Dali raboti vyobste kakto trqbva tozi CAN - SIT1050T? Ako ne -> MCP2551!"
- note removed: "Ako ima nuzda ot GPIO-ta, moze da se pomisli dali da ne izvedem i\nHDMI_INT i HDMI_RSTN systo na extensionite!?"
- note removed: "Da se proveri dali extensions sa syvmestimi s Lime2!!!"
