File: HARDWARE/STMP157-OLinuXino-LIME2/1. Latest hardware revision/STMP157-OLinuXino-LIME2_Rev_B1/eMMC, SPI-Flash, T-Card and Boot.sch (KiCad schematic (older format))
At the start: 34 parts, among them Q1 Q32.768kHz/12.5pF/2P/SMD1206, U1 STM32MP157CAA3x

Commit message: 3d view components fixed
Parts:
- BOOT0_VDD1, BOOT1_VDD1, BOOT2_VDD1: symbol OLIMEX_Jumpers:SJ -> STMP157-OLinuXino-LIME2_Rev_B1:SJ
- C127, C40, C41, C42, C43, C46: symbol OLIMEX_RCL:C -> STMP157-OLinuXino-LIME2_Rev_B1:C
- CR1: symbol OLIMEX_Devices:Oscillator-100MHZ_TXC-7W -> STMP157-OLinuXino-LIME2_Rev_B1:Oscillator-100MHZ_TXC-7W
- D5: symbol OLIMEX_Diodes:D_Schottky -> STMP157-OLinuXino-LIME2_Rev_B1:D_Schottky
- FID1, FID2, FID3, FID4, FID5, FID6: symbol OLIMEX_OTHER:Fiducial -> STMP157-OLinuXino-LIME2_Rev_B1:Fiducial
- Flash_Con1: symbol OLIMEX_Connectors:Flash_Con[DF12(3.0)-40DS-0.5V(86)] -> STMP157-OLinuXino-LIME2_Rev_B1:Flash_Con[DF12(3.0)-40DS-0.5V(86)]
- L1: symbol OLIMEX_RCL:L -> STMP157-OLinuXino-LIME2_Rev_B1:L
- MICRO_SD1: symbol OLIMEX_Connectors:MICRO_SD(TFC-WPAPR-08) -> STMP157-OLinuXino-LIME2_Rev_B1:MICRO_SD(TFC-WPAPR-08)
- Q1: symbol OLIMEX_Devices:Crystal -> STMP157-OLinuXino-LIME2_Rev_B1:Crystal
- R139, R40, R43, R46, R48, R49, R50, R51, R53, R54, R55: symbol OLIMEX_RCL:R -> STMP157-OLinuXino-LIME2_Rev_B1:R
- RM1: symbol OLIMEX_RCL:RA1206_(4x0603)_4B8_Smashed -> STMP157-OLinuXino-LIME2_Rev_B1:RA1206_(4x0603)_4B8_Smashed
- U1: symbol OLIMEX_IC:STM32MP157CAA3x -> STMP157-OLinuXino-LIME2_Rev_B1:STM32MP157CAA3x
Other:
- note removed: "Notes:\n=====\n1. NRST and NRST_CORE are separated in all schematics, but are connected together in AN5256, \ni.e. "STM32MP157 discrete power supply hardware integration" (see: en.DM00561921.pdf/page 10).\nKoe e vqrnoto v krajna smetka??? V datasheet pishe, 4e NRST_CORE ima "permanent pull-up resistor, R PU" okolo 40k OHm\n2. "Adding an external resistor between OSC32_IN and OSC32_OUT is forbidde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"
