File: HARDWARE/A10-OLinuXino-LIME/3. Templates and more/A10-OLinuXino-LIME revision B SHIELD TEMPLATE KiCAD/A10_OLinuXino_Lime_Rev-B_SHIELD_TEMPLATE.sch (KiCad schematic (older format))
At the start: 5 parts

Commit message: Update
Parts:
- GPIO-1, GPIO-2, GPIO-3, LCD_CON1: symbol FL40YA-V36P-2X20-LF -> A10_OLinuXino_Lime_Rev-B_SHIELD_TEMPLATE:FL40YA-V36P-2X20-LF
- GPIO-4: symbol FL20YA-V36P-2X10-LF -> A10_OLinuXino_Lime_Rev-B_SHIELD_TEMPLATE:FL20YA-V36P-2X10-LF
Connections:
- wire segments 191 -> 193
Changed lines of the file:
@@
-EESchema Schematic File Version 2
-LIBS:A10-OLinuXino-Lime_Rev-B_SHIELD_TEMPLATE_-cache
-LIBS:A10_OLIMEXINO_LIME_SHIELD_1
-LIBS:power
-EELAYER 27 0
+EESchema Schematic File Version 4
+LIBS:A10_OLinuXino_Lime_Rev-B_SHIELD_TEMPLATE-cache
+EELAYER 29 0
 EELAYER END
 $Descr B 17000 11000
@@
 	6700 5100 9200 5100
 Wire Wire Line
-	6700 8000 7500 8000
+	6700 8000 6900 8000
 Wire Wire Line
 	6700 8100 6900 8100
@@
 Connection ~ 6900 8000
 Wire Wire Line
-	14000 5100 15000 5100
+	14000 5100 14200 5100
 Wire Wire Line
 	14000 5200 14200 5200
@@
 YP_TP
 $Comp
-L FL20YA-V36P-2X10-LF GPIO-4
+L A10_OLinuXino_Lime_Rev-B_SHIELD_TEMPLATE:FL20YA-V36P-2X10-LF GPIO-4
 U 1 1 52FC8278
 P 13650 3500
@@
 $EndComp
 $Comp
-L FL40YA-V36P-2X20-LF GPIO-3
+L A10_OLinuXino_Lime_Rev-B_SHIELD_TEMPLATE:FL40YA-V36P-2X20-LF GPIO-3
 U 1 1 52FC87FB
 P 6350 9000
@@
 $EndComp
 $Comp
-L FL40YA-V36P-2X20-LF GPIO-2
+L A10_OLinuXino_Lime_Rev-B_SHIELD_TEMPLATE:FL40YA-V36P-2X20-LF GPIO-2
 U 1 1 52FC9419
 P 6350 6100
@@
 $EndComp
 $Comp
-L FL40YA-V36P-2X20-LF GPIO-1
+L A10_OLinuXino_Lime_Rev-B_SHIELD_TEMPLATE:FL40YA-V36P-2X20-LF GPIO-1
 U 1 1 52FC941F
 P 6350 3300
@@
 $EndComp
 $Comp
-L FL40YA-V36P-2X20-LF LCD_CON1
+L A10_OLinuXino_Lime_Rev-B_SHIELD_TEMPLATE:FL40YA-V36P-2X20-LF LCD_CON1
 U 1 1 52FC94E5
 P 13650 6100
@@
 $EndComp
 $Comp
-L +5V #PWR01
+L A10_OLinuXino_Lime_Rev-B_SHIELD_TEMPLATE:+5V #PWR01
 U 1 1 52FCA551
 P 4800 2100
 F 0 "#PWR01" H 4800 2190 20  0001 C CNN
-F 1 "+5V" H 4800 2190 30  0000 C CNN
+F 1 "+5V" H 4800 2275 50  0000 C CNN
 F 2 "" H 4800 2100 60  0000 C CNN
 F 3 "" H 4800 2100 60  0000 C CNN
@@
 $EndComp
 $Comp
-L +3.3V #PWR02
-U 1 1 52FCA570
-P 4600 2100
-F 0 "#PWR02" H 4600 2060 30  0001 C CNN
-F 1 "+3.3V" H 4600 2210 30  0000 C CNN
-F 2 "" H 4600 2100 60  0000 C CNN
-F 3 "" H 4600 2100 60  0000 C CNN
-	1    4600 2100
-	1    0    0    -1
-$EndComp
-$Comp
-L +5V #PWR03
+L A10_OLinuXino_Lime_Rev-B_SHIELD_TEMPLATE:+5V #PWR03
 U 1 1 52FCA5EE
 P 4800 4900
 F 0 "#PWR03" H 4800 4990 20  0001 C CNN
-F 1 "+5V" H 4800 4990 30  0000 C CNN
+F 1 "+5V" H 4800 5075 50  0000 C CNN
 F 2 "" H 4800 4900 60  0000 C CNN
 F 3 "" H 4800 4900 60  0000 C CNN
@@
 $EndComp
 $Comp
-L +3.3V #PWR04
-U 1 1 52FCA5FD
-P 4600 4900
-F 0 "#PWR04" H 4600 4860 30  0001 C CNN
-F 1 "+3.3V" H 4600 5010 30  0000 C CNN
-F 2 "" H 4600 4900 60  0000 C CNN
-F 3 "" H 4600 4900 60  0000 C CNN
-	1    4600 4900
-	1    0    0    -1
-$EndComp
-$Comp
-L +5V #PWR05
+L A10_OLinuXino_Lime_Rev-B_SHIELD_TEMPLATE:+5V #PWR05
 U 1 1 52FCA63E
 P 4800 7800
 F 0 "#PWR05" H 4800 7890 20  0001 C CNN
-F 1 "+5V" H 4800 7890 30  0000 C CNN
+F 1 "+5V" H 4825 7975 50  0000 C CNN
 F 2 "" H 4800 7800 60  0000 C CNN
 F 3 "" H 4800 7800 60  0000 C CNN
@@
 $EndComp
 $Comp
-L +3.3V #PWR06
-U 1 1 52FCA64D
-P 12100 2800
-F 0 "#PWR06" H 12100 2760 30  0001 C CNN
-F 1 "+3.3V" H 12100 2910 30  0000 C CNN
-F 2 "" H 12100 2800 60  0000 C CNN
-F 3 "" H 12100 2800 60  0000 C CNN
-	1    12100 2800
-	1    0    0    -1
-$EndComp
-$Comp
-L +3.3V #PWR07
-U 1 1 52FCA65C
-P 12200 4900
-F 0 "#PWR07" H 12200 4860 30  0001 C CNN
-F 1 "+3.3V" H 12200 5010 30  0000 C CNN
-F 2 "" H 12200 4900 60  0000 C CNN
-F 3 "" H 12200 4900 60  0000 C CNN
-	1    12200 4900
-	1    0    0    -1
-$EndComp
-$Comp
-L +5V #PWR08
+L A10_OLinuXino_Lime_Rev-B_SHIELD_TEMPLATE:+5V #PWR08
 U 1 1 52FCA66B
 P 12400 4900
 F 0 "#PWR08" H 12400 4990 20  0001 C CNN
-F 1 "+5V" H 12400 4990 30  0000 C CNN
+F 1 "+5V" H 12400 5075 50  0000 C CNN
 F 2 "" H 12400 4900 60  0000 C CNN
 F 3 "" H 12400 4900 60  0000 C CNN
@@
 $EndComp
 $Comp
-L GND #PWR09
+L A10_OLinuXino_Lime_Rev-B_SHIELD_TEMPLATE:GND #PWR09
 U 1 1 52FCA67A
 P 9300 2300
@@
 $EndComp
 $Comp
-L GNDPWR #PWR010
+L A10_OLinuXino_Lime_Rev-B_SHIELD_TEMPLATE:GNDPWR #PWR010
 U 1 1 52FCA698
 P 9100 2400
 F 0 "#PWR010" H 9100 2450 40  0001 C CNN
-F 1 "GNDPWR" H 9100 2320 40  0000 C CNN
+F 1 "GNDPWR" V 9100 2150 40  0001 C CNN
 F 2 "" H 9100 2400 60  0000 C CNN
 F 3 "" H 9100 2400 60  0000 C CNN
@@
 $EndComp
 $Comp
-L GND #PWR011
+L A10_OLinuXino_Lime_Rev-B_SHIELD_TEMPLATE:GND #PWR011
 U 1 1 52FCA6A7
 P 9200 5100
@@
 $EndComp
 $Comp
-L GND #PWR012
+L A10_OLinuXino_Lime_Rev-B_SHIELD_TEMPLATE:GND #PWR012
 U 1 1 52FCA6B6
 P 7500 8000
@@
 $EndComp
 $Comp
-L GND #PWR013
+L A10_OLinuXino_Lime_Rev-B_SHIELD_TEMPLATE:GND #PWR013
 U 1 1 52FCA6C5
 P 15800 3100
@@
 $EndComp
 $Comp
-L GND #PWR014
+L A10_OLinuXino_Lime_Rev-B_SHIELD_TEMPLATE:GND #PWR014
 U 1 1 52FCA6D4
 P 15000 5100
@@
 	0    -1   -1   0
 $EndComp
+Wire Wire Line
+	6900 8000 7500 8000
+Wire Wire Line
+	14200 5100 15000 5100
+$Comp
+L A10_OLinuXino_Lime_Rev-B_SHIELD_TEMPLATE:+3.3V #PWR?
+U 1 1 62AD6413
+P 4600 7800
+F 0 "#PWR?" H 4600 7650 50  0001 C CNN
+F 1 "+3.3V" H 4600 7975 50  0000 C CNN
+F 2 "" H 4600 7800 60  0000 C CNN
+F 3 "" H 4600 7800 60  0000 C CNN
+	1    4600 7800
+	1    0    0    -1
+$EndComp
+$Comp
+L A10_OLinuXino_Lime_Rev-B_SHIELD_TEMPLATE:+3.3V #PWR?
+U 1 1 62AD6C54
+P 4600 4900
+F 0 "#PWR?" H 4600 4750 50  0001 C CNN
+F 1 "+3.3V" H 4550 5075 50  0000 C CNN
+F 2 "" H 4600 4900 60  0000 C CNN
+F 3 "" H 4600 4900 60  0000 C CNN
+	1    4600 4900
+	1    0    0    -1
+$EndComp
+$Comp
+L A10_OLinuXino_Lime_Rev-B_SHIELD_TEMPLATE:+3.3V #PWR?
+U 1 1 62AD7347
+P 4600 2100
+F 0 "#PWR?" H 4600 1950 50  0001 C CNN
+F 1 "+3.3V" H 4550 2275 50  0000 C CNN
+F 2 "" H 4600 2100 60  0000 C CNN
+F 3 "" H 4600 2100 60  0000 C CNN
+	1    4600 2100
+	1    0    0    -1
+$EndComp
+$Comp
+L A10_OLinuXino_Lime_Rev-B_SHIELD_TEMPLATE:+3.3V #PWR?
+U 1 1 62AD7ACF
+P 12100 2800
+F 0 "#PWR?" H 12100 2650 50  0001 C CNN
+F 1 "+3.3V" H 12115 2973 50  0000 C CNN
+F 2 "" H 12100 2800 60  0000 C CNN
+F 3 "" H 12100 2800 60  0000 C CNN
+	1    12100 2800
+	1    0    0    -1
+$EndComp
+$Comp
+L A10_OLinuXino_Lime_Rev-B_SHIELD_TEMPLATE:+3.3V #PWR?
+U 1 1 62AD84CC
+P 12200 4900
+F 0 "#PWR?" H 12200 4750 50  0001 C CNN
+F 1 "+3.3V" H 12175 5075 50  0000 C CNN
+F 2 "" H 12200 4900 60  0000 C CNN
+F 3 "" H 12200 4900 60  0000 C CNN
+	1    12200 4900
+	1    0    0    -1
+$EndComp
 $EndSCHEMATC
